Commit message: the training works

File: sim/stompy_legs/robot_fixed.urdf (robot description, URDF)
Before this commit: robot lower_limbs, 46 links, 45 joints
Joints:
- joint left ankle pitch: limit lower=-0.8 upper=0.6 effort=24 velocity=12 -> lower=-0.8 upper=0.6 effort=80 velocity=5
- joint left ankle roll: limit lower=1 upper=2.3 effort=24 velocity=12 -> lower=1 upper=2.3 effort=80 velocity=5
- joint left hip pitch: limit lower=0.5 upper=2.69 effort=150 velocity=25 -> lower=0.5 upper=2.69 effort=150 velocity=5
- joint left hip roll: limit lower=-0.5 upper=0.5 effort=90 velocity=25 -> lower=-0.5 upper=0.5 effort=90 velocity=5
- joint left hip yaw: limit lower=0.5 upper=1.19 effort=90 velocity=25 -> lower=0.5 upper=1.19 effort=90 velocity=5
- joint left knee pitch: limit lower=0.5 upper=2.5 effort=90 velocity=25 -> lower=0.5 upper=2.5 effort=90 velocity=5
- joint right ankle pitch: limit lower=0 upper=1.5 effort=24 velocity=12 -> lower=0 upper=1.5 effort=80 velocity=5
- joint right ankle roll: limit lower=1 upper=2.3 effort=24 velocity=12 -> lower=1 upper=2.3 effort=80 velocity=5
- joint right hip pitch: limit lower=-1 upper=1 effort=150 velocity=25 -> lower=-1 upper=1 effort=150 velocity=5
- joint right hip roll: limit lower=-2.39 upper=-1 effort=90 velocity=25 -> lower=-2.39 upper=-1 effort=90 velocity=5
- joint right hip yaw: limit lower=-2.2 upper=-1 effort=90 velocity=25 -> lower=-2.3 upper=-1.76 effort=90 velocity=5
- joint right knee pitch: limit lower=2.09 upper=3.2 effort=90 velocity=25 -> lower=2.09 upper=3.2 effort=90 velocity=5

Commit message: sort of behaves, doest move forward but not backward either

File: sim/stompy_legs/robot_fixed.urdf (robot description, URDF)
Before this commit: robot lower_limbs, 46 links, 45 joints
Joints:
- joint left ankle pitch: limit lower=-0.8 upper=0.6 effort=80 velocity=5 -> lower=-0.8 upper=0.6 effort=100 velocity=12
- joint left ankle roll: limit lower=1 upper=2.3 effort=80 velocity=5 -> lower=1 upper=2.3 effort=100 velocity=12
- joint left hip pitch: limit lower=0.5 upper=2.69 effort=150 velocity=5 -> lower=0.5 upper=2.69 effort=250 velocity=12
- joint left hip roll: limit lower=-0.5 upper=0.5 effort=90 velocity=5 -> lower=-0.5 upper=0.5 effort=250 velocity=12
- joint left hip yaw: limit lower=0.5 upper=1.19 effort=90 velocity=5 -> lower=0.5 upper=1.19 effort=250 velocity=12
- joint left knee pitch: limit lower=0.5 upper=2.5 effort=90 velocity=5 -> lower=0.5 upper=2.5 effort=250 velocity=12
- joint right ankle pitch: limit lower=0 upper=1.5 effort=80 velocity=5 -> lower=0 upper=1.5 effort=100 velocity=12
- joint right ankle roll: limit lower=1 upper=2.3 effort=80 velocity=5 -> lower=1 upper=2.3 effort=100 velocity=12
- joint right hip pitch: limit lower=-1 upper=1 effort=150 velocity=5 -> lower=-1 upper=1 effort=250 velocity=12
- joint right hip roll: limit lower=-2.39 upper=-1 effort=90 velocity=5 -> lower=-2.39 upper=-1 effort=250 velocity=12
- joint right hip yaw: limit lower=-2.3 upper=-1.76 effort=90 velocity=5 -> lower=-2.3 upper=-1.76 effort=250 velocity=12
- joint right knee pitch: limit lower=2.09 upper=3.2 effort=90 velocity=5 -> lower=2.09 upper=3.2 effort=250 velocity=12

Commit message: current setup makes the robot learns to walk reliably but sideways

File: sim/stompy_legs/robot_fixed.urdf (robot description, URDF)
Before this commit: robot lower_limbs, 46 links, 45 joints
Joints:
- joint left ankle pitch: limit lower=-0.8 upper=0.6 effort=100 velocity=12 -> lower=-0.8 upper=0.6 effort=24 velocity=24
- joint left ankle roll: limit lower=1 upper=2.3 effort=100 velocity=12 -> lower=1 upper=2.3 effort=24 velocity=24
- joint left hip pitch: limit lower=0.5 upper=2.69 effort=250 velocity=12 -> lower=0.5 upper=2.69 effort=150 velocity=25
- joint left hip roll: limit lower=-0.5 upper=0.5 effort=250 velocity=12 -> lower=-0.5 upper=0.5 effort=90 velocity=25
- joint left hip yaw: limit lower=0.5 upper=1.19 effort=250 velocity=12 -> lower=0.5 upper=1.19 effort=90 velocity=25
- joint left knee pitch: limit lower=0.5 upper=2.5 effort=250 velocity=12 -> lower=0.5 upper=2.5 effort=90 velocity=25
- joint right ankle pitch: limit lower=0 upper=1.5 effort=100 velocity=12 -> lower=0 upper=1.5 effort=24 velocity=24
- joint right ankle roll: limit lower=1 upper=2.3 effort=100 velocity=12 -> lower=1 upper=2.3 effort=24 velocity=24
- joint right hip pitch: limit lower=-1 upper=1 effort=250 velocity=12 -> lower=-1 upper=1 effort=150 velocity=25
- joint right hip roll: limit lower=-2.39 upper=-1 effort=250 velocity=12 -> lower=-2.39 upper=-1 effort=90 velocity=25
- joint right hip yaw: limit lower=-2.3 upper=-1.76 effort=250 velocity=12 -> lower=-2.6 upper=-1.5 effort=90 velocity=25
- joint right knee pitch: limit lower=2.09 upper=3.2 effort=250 velocity=12 -> lower=2.09 upper=3.2 effort=90 velocity=25
