Commit message: add solidworks model, errors on observation

File: sim/stompy_legs/robot.urdf (robot description, URDF)
Before this commit: robot lower_limbs, 46 links, 45 joints
Links:
- added link link_part_1_1, mass 0.001; collision mesh filename=./meshes/part_1_1_simple.stl; visual mesh filename=./meshes/part_1_1_simple.stl
- link link_leg_assembly_left_1_rmd_x12_150_mock_1_inner_x12_150_1: mass 0.023817612 -> 0.1494739
- link link_leg_assembly_left_1_rmd_x12_150_mock_1_outer_x12_150_1: mass 0.18332765 -> 1.1505225
- link link_leg_assembly_right_1_rmd_x12_150_mock_1_inner_x12_150_1: mass 0.023817612 -> 0.1494739
- link link_leg_assembly_right_1_rmd_x12_150_mock_1_outer_x12_150_1: mass 0.18332765 -> 1.1505225
Joints:
- added joint joint_fastened_10: type fixed, parent link_leg_assembly_left_1_leg_part_1_2, child link_part_1_1, origin xyz=0.02779169 -0.048790465 0.050524107 rpy=3.1415927 0 -1.5707963
- joint left ankle pitch: limit lower=-0.8 upper=0.6 effort=80 velocity=5 -> lower=-1.5707963 upper=2.1816616 effort=24 velocity=5
- joint left ankle roll: limit lower=1 upper=5 effort=80 velocity=5 -> lower=-2.268928 upper=-1.2217305 effort=24 velocity=5
- joint left hip pitch: limit lower=0.25 upper=2.69 effort=80 velocity=5 -> lower=-4.712389 upper=4.712389 effort=80 velocity=5
- joint left hip roll: limit lower=-0.5 upper=0.5 effort=80 velocity=5 -> lower=-3.1415927 upper=0 effort=90 velocity=5
- joint left hip yaw: limit lower=0.5 upper=1.19 effort=80 velocity=5 -> lower=-1.0471976 upper=2.0943951 effort=90 velocity=5
- joint left knee pitch: limit lower=0.5 upper=2.5 effort=80 velocity=5 -> lower=-4.712389 upper=4.712389 effort=90 velocity=5
- joint right ankle pitch: limit lower=0 upper=1.5 effort=80 velocity=5 -> lower=-1.5707963 upper=2.1816616 effort=24 velocity=5
- joint right ankle roll: limit lower=1 upper=2.3 effort=80 velocity=5 -> lower=-2.268928 upper=-1.2217305 effort=24 velocity=5
- joint right hip pitch: limit lower=-1 upper=1.25 effort=80 velocity=5 -> lower=-4.712389 upper=4.712389 effort=80 velocity=5
- joint right hip roll: limit lower=-2.39 upper=-1 effort=80 velocity=5 -> lower=-3.1415927 upper=3.1415927 effort=90 velocity=5
- joint right hip yaw: limit lower=-2.2 upper=-1 effort=80 velocity=5 -> lower=-4.712389 upper=4.712389 effort=90 velocity=5
- joint right knee pitch: limit lower=1.54 upper=3.5 effort=80 velocity=5 -> lower=-4.712389 upper=4.712389 effort=90 velocity=5

File: sim/stompy_legs/robot_fixed.urdf (robot description, URDF)
Before this commit: robot lower_limbs, 46 links, 45 joints
Links:
- added link link_part_1_1, mass 0.001; collision mesh filename=./meshes/part_1_1_simple.stl; visual mesh filename=./meshes/part_1_1_simple.stl
- link link_leg_assembly_left_1_rmd_x12_150_mock_1_inner_x12_150_1: mass 0.023817612 -> 0.1494739
- link link_leg_assembly_left_1_rmd_x12_150_mock_1_outer_x12_150_1: mass 0.18332765 -> 1.1505225
- link link_leg_assembly_right_1_rmd_x12_150_mock_1_inner_x12_150_1: mass 0.023817612 -> 0.1494739
- link link_leg_assembly_right_1_rmd_x12_150_mock_1_outer_x12_150_1: mass 0.18332765 -> 1.1505225
Joints:
- added joint joint_fastened_10: type fixed, parent link_leg_assembly_left_1_leg_part_1_2, child link_part_1_1, origin xyz=0.02779169 -0.048790465 0.050524107 rpy=3.1415927 0 -1.5707963
- joint left hip pitch: limit lower=0.5 upper=2.69 effort=150 velocity=25 -> lower=0.5 upper=2.69 effort=150 velocity=40
- joint left hip roll: limit lower=-0.5 upper=0.5 effort=90 velocity=25 -> lower=0.05 upper=0.15 effort=90 velocity=40
- joint left hip yaw: limit lower=0.5 upper=1.19 effort=90 velocity=25 -> lower=0.98 upper=1.08 effort=90 velocity=40
- joint left knee pitch: limit lower=0.5 upper=2.5 effort=90 velocity=25 -> lower=0.5 upper=2.5 effort=90 velocity=40
- joint right hip pitch: limit lower=-1 upper=1 effort=150 velocity=25 -> lower=-1 upper=1 effort=150 velocity=40
- joint right hip roll: limit lower=-2.39 upper=-1 effort=90 velocity=25 -> lower=-1.63 upper=-1.57 effort=90 velocity=40
- joint right hip yaw: limit lower=-2.6 upper=-1.5 effort=90 velocity=25 -> lower=-2.2 upper=-2.1 effort=90 velocity=40
- joint right knee pitch: limit lower=2.09 upper=3.2 effort=90 velocity=25 -> lower=2.09 upper=3.2 effort=90 velocity=40
