Commit message: saving working but not perfect setup

File: sim/new_stompy/robot_fixed.urdf (robot description, URDF)
Before this commit: robot stompy, 42 links, 41 joints
Joints:
- joint Foot motor fixed: limit lower=-0.45 upper=0.45 effort=0 velocity=0 -> lower=-0.45 upper=0.45 effort=24 velocity=24
- joint Knee motor inner: limit lower=-1.57 upper=0 effort=0 velocity=0 -> lower=-1.57 upper=0 effort=90 velocity=40
