Commit message: saving dora calibration setup

File: sim/resources/stompymini/robot_fixed.urdf (robot description, URDF)
Before this commit: robot full_assembly, 253 links, 252 joints
Links:
- link link_lower_half_assembly_1_left_leg_1_knee_left_1: mass 0.82466495 -> 0.082466495
- link link_lower_half_assembly_1_left_leg_1_robstride_01_mock_1_rs_01_stator_1: mass 0.34790535 -> 0.034790535
- link link_lower_half_assembly_1_left_leg_1_robstride_04_mock_1_rs_04_rotor_1: mass 0.18007617 -> 0.018007617
- link link_lower_half_assembly_1_right_leg_1_hip_roll_right_rear_1: mass 0.97382295 -> 0.097382295
Joints:
- joint left ankle pitch: limit lower=-2.8 upper=-0.8 effort=17 velocity=40 -> lower=-8 upper=8 effort=17 velocity=40
- joint left hip pitch: limit lower=-1.28 upper=0.72 effort=120 velocity=40 -> lower=-8 upper=72 effort=120 velocity=40
- joint left hip roll: limit lower=0.5 upper=2.5 effort=17 velocity=40 -> lower=-5 upper=5 effort=17 velocity=40
- joint left hip yaw: limit lower=0.62 upper=2.62 effort=120 velocity=40 -> lower=-6 upper=6 effort=120 velocity=40
- joint right ankle pitch: limit lower=-0.58 upper=1.42 effort=17 velocity=40 -> lower=-8 upper=4 effort=17 velocity=40
- joint right hip pitch: limit lower=2.55 upper=4.55 effort=120 velocity=40 -> lower=-2.55 upper=6 effort=120 velocity=40
- joint right hip roll: limit lower=2.18 upper=4.18 effort=17 velocity=40 -> lower=-2.18 upper=48 effort=17 velocity=40
- joint right hip yaw: limit lower=2.24 upper=4.24 effort=120 velocity=40 -> lower=-2.24 upper=24 effort=120 velocity=40
